File: 860.sch (KiCad schematic (older format))
At the start: 150 parts, among them J1 PJ301B, J2 PJ301B, J3 PJ301B, J4 PJ301B, J5 PJ301B, J6 PJ301B, P1 CONN_02X05, Q1 BCM857BS, Q2 BCM857BS, Q3 J112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

Commit message: routed, silk screen adjusted
Parts:
- C18, C25, C6, C7: footprint MyModules:SM0805-HAND -> MyModules:SM0805-HAND-C
Changed lines of the file:
@@
 F 0 "C6" H 8325 12275 50  0000 L CNN
 F 1 "330pF" H 8325 12075 50  0000 L CNN
-F 2 "MyModules:SM0805-HAND" H 8275 12175 60  0001 C CNN
+F 2 "MyModules:SM0805-HAND-C" H 8275 12175 60  0001 C CNN
 F 3 "" H 8275 12175 60  0000 C CNN
 	1    8275 12175
@@
 F 0 "C7" H 10925 12275 50  0000 L CNN
 F 1 "330pF" H 10925 12075 50  0000 L CNN
-F 2 "MyModules:SM0805-HAND" H 10875 12175 60  0001 C CNN
+F 2 "MyModules:SM0805-HAND-C" H 10875 12175 60  0001 C CNN
 F 3 "" H 10875 12175 60  0000 C CNN
 	1    10875 12175
@@
 F 0 "C18" H 16625 12275 50  0000 L CNN
 F 1 "330pF" H 16625 12075 50  0000 L CNN
-F 2 "MyModules:SM0805-HAND" H 16575 12175 60  0001 C CNN
+F 2 "MyModules:SM0805-HAND-C" H 16575 12175 60  0001 C CNN
 F 3 "" H 16575 12175 60  0000 C CNN
 	1    16575 12175
@@
 F 0 "C25" H 19225 12275 50  0000 L CNN
 F 1 "330pF" H 19225 12075 50  0000 L CNN
-F 2 "MyModules:SM0805-HAND" H 19175 12175 60  0001 C CNN
+F 2 "MyModules:SM0805-HAND-C" H 19175 12175 60  0001 C CNN
 F 3 "" H 19175 12175 60  0000 C CNN
 	1    19175 12175
